File: STM32F446/KiCad/Inverter F446.kicad_sch (KiCad schematic)
At the start: 103 parts, among them J1 Screw_Terminal_01x02, J2 Screw_Terminal_01x03, Q1 BC547, Q2 BC557, Q3 BC547, Q4 BC547, Q5 BC557, Q6 BC547, Q7 BC547, Q8 BC557, Q9 BC547, U1 NUCLEO-F446RE, U2 INA181, U3 INA181, U4 INA181, U5 MCP6004

Commit message: PCB makeing
Parts:
- added C31, C32: 1µF, Capacitor_THT:C_Disc_D7.5mm_W5.0mm_P5.00mm, symbol Device:C
- added R33, R34, R35: 3k3, Resistor_THT:R_Axial_DIN0207_L6.3mm_D2.5mm_P10.16mm_Horizontal, symbol Device:R
- added unit 2 of U1
- added unit 6 of U1
- added unit 5 of U1
- added unit 3 of U1
- added unit 4 of U1
- R11, R12, R20, R21, R25, R26: value 1k -> 3k3
Connections:
- net OffsetVoltage is gone; now on net OffsetV: R16.1, R22.1, R27.1, U5.1, U5.2 (-)
- net +5V: no longer R13.2
- net Current_Phase_1: now also R33.2
- net Current_Phase_2: now also R34.2, R35.2
- net GND: now also U1.CN7_19 (CN7_GND), U1.CN7_20 (CN7_GND), U1.CN7_22 (CN7_GND), U1.CN7_8 (CN7_GND), C31.2, C32.2, R33.1, R34.1, R35.1, U1.CN10_20 (CN10_GND), U1.CN10_9 (CN10_GND), U1.CN5_7 (CN5_GND), U1.CN6_6 (CN6_GND), U1.CN6_7 (CN6_GND)
- net Phase1: now also U2.4 (-), U4.4 (-); no longer U2.3 (+), U4.3 (+)
- net Phase2: now also U3.4 (-); no longer U3.3 (+)
- net at L11.2, R15.1: now also U3.3 (+); no longer U3.4 (-)
- net at L4.2, R10.1: now also U2.3 (+); no longer U2.4 (-)
- net at L16.2, R18.1: now also U4.3 (+); no longer U4.4 (-)
- net +3.3V: now reaches U1.CN7_16 (CN7_+3V3)
- net +3.3V: now also R13.2, U1.CN6_4 (CN6_+3V3)
- net at U1.CN7_6 (E5V): now also C31.1, C32.1
- net HalfVcc renamed OffsetV
- new net TIM_CH1: U1.CN10_23 (PA8)
- new net TIM_CH1N: U1.CN10_30 (PB13)
- new net TIM_CH2: U1.CN10_21 (PA9)
- new net TIM_CH2N: U1.CN10_28 (PB14)
- new net TIM_CH3: U1.CN10_33 (PA10)
- new net TIM_CH3N: U1.CN10_26 (PB15)
Other:
- moved on the sheet: C17, C19, C20, C21, C22, C24, C28, C29, C30, J2, R30, R31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

Commit message: PCB Placement Done
Parts:
- removed L5: 1mH, Inductor_THT:L_Axial_L12.0mm_D5.0mm_P15.24mm_Horizontal_Fastron_MISC, symbol Device:L
- added C33: 220µF, Capacitor_THT:CP_Radial_D8.0mm_P5.00mm, symbol Device:C
- added C34: 1µF, Capacitor_THT:C_Disc_D7.5mm_W5.0mm_P5.00mm, symbol Device:C
- added R36, R37: 3k3, Resistor_THT:R_Axial_DIN0207_L6.3mm_D2.5mm_P10.16mm_Horizontal, symbol Device:R
- added R38, R39, R40: 1.5, Resistor_THT:R_Axial_DIN0207_L6.3mm_D2.5mm_P10.16mm_Horizontal, symbol Device:R
- C32: value 1µF -> 100µF; footprint Capacitor_THT:C_Disc_D7.5mm_W5.0mm_P5.00mm -> Capacitor_THT:CP_Radial_D6.3mm_P2.50mm
- R10, R15, R18: value 1 -> 1.5
- R13, R14: value 1k -> 3k3
Connections:
- net Current_Phase_1 is gone; now on net ADC1_IN11: C28.1, R30.1, R33.2
- net OffsetV is gone; now on net ADC1_IN4: C19.1, C21.1, C24.1, R16.1, R22.1, R27.1, U2.5 (REF), U3.5 (REF), U4.5 (REF), U5.1, U5.2 (-)
- net +5V: now also J1.2 (Pin_2), Q2.3 (E), Q5.3 (E), Q8.3 (E), C33.1, R36.2; no longer Q2.1 (C), Q5.1 (C), Q8.1 (C)
- net GND: now also C33.2, C34.2, R37.1
- net Phase1: now also U2.3 (+), R38.2; no longer R18.2, U2.4 (-), U4.4 (-)
- net Phase2: now also U3.3 (+), R39.2; no longer U3.4 (-)
- net Phase3: now also R18.2, U4.3 (+), R40.2
- net TIM_CH1: now also R2.1
- net TIM_CH1N: now also R3.1
- net TIM_CH2: now also R4.1
- net TIM_CH2N: now also R5.1
- net TIM_CH3: now also R7.1
- net TIM_CH3N: now also R8.1
- net at L11.2, R15.1: now also U3.4 (-), R39.1; no longer U3.3 (+)
- net at L4.2, R10.1: now also U2.4 (-), R38.1; no longer U2.3 (+)
- net at D1.2 (A), D3.1 (K), L6.1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: now also Q2.1 (C); no longer Q2.3 (E)
- net ADC2_IN6: now reaches U1.CN10_13 (PA6)
- net ADC2_IN6: now also C34.1, R36.1, R37.2
- net at L16.2, R18.1: now also U4.4 (-), R40.1; no longer U4.3 (+)
- net at D5.2 (A), D6.1 (K), L7.1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: now also Q5.1 (C); no longer Q5.3 (E)
- net at D8.2 (A), D9.1 (K), L12.1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: now also Q8.1 (C); no longer Q8.3 (E)
- net ADC3_IN0: now reaches U1.CN7_28 (PA0)
- net ADC3_IN0: now also C27.1, R29.2
- net ADC3_IN1: now reaches U1.CN7_30 (PA1)
- net ADC3_IN1: now also C30.1, R32.1, R35.2
- net ADC1_IN4: now reaches U1.CN7_32 (PA4)
- net ADC2_IN12: now reaches U1.CN7_35 (PC2)
- net ADC2_IN12: now also C26.1, R24.2
- net ADC1_IN11: now reaches U1.CN7_36 (PC1/PB9)
- net ADC2_IN13: now reaches U1.CN7_37 (PC3)
- net ADC2_IN13: now also C29.1, R31.1, R34.2
- net ADC1_IN10: now reaches U1.CN7_38 (PC0/PB8)
- net ADC1_IN10: now also C25.1, R19.2
- removed net Current_Phase_2: C29.1, C30.1, R31.1, R32.1, R34.2, R35.2
- removed net Ph1-2_ADC: C25.1, C26.1, C27.1, R19.2, R24.2, R29.2
Other:
- note added: "Micro Controller"
- moved on the sheet: C17, C18, C19, C20, C21, C22, C23, C24, C28, C29, C30, C31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

Commit message: A bit of clean-up
Parts:
- removed R33, R34, R35: 3k3, Resistor_THT:R_Axial_DIN0207_L6.3mm_D2.5mm_P10.16mm_Horizontal, symbol Device:R
- R16, R17, R22, R23, R27, R28: value 1k -> 510
Other:
- note added: "((1.5ohm/2)*I_out)*20 + 1.65V = V_out (0.15V to 3.15V)"
- note added: "((510ohm/3.3kohm)*V_diff) + 1.65V = V_out (0.1V to 3.2V)"
- moved on the sheet: C28, C29, C30
