File: STM32F446/KiCad/Inverter F446.kicad_pcb (KiCad board)
At the start: 2 copper layers, 103 parts, among them J1 Screw_Terminal_01x02, J2 Screw_Terminal_01x03, Q1 BC547, Q2 BC557, Q3 BC547, Q4 BC547, Q5 BC557, Q6 BC547, Q7 BC547, Q8 BC557, Q9 BC547, U1 NUCLEO-F446RE, U2 INA181, U3 INA181, U4 INA181, U5 MCP6004

Commit message: PCB Placement Done
Parts:
- removed L5: 1mH, Inductor_THT:L_Axial_L12.0mm_D5.0mm_P15.24mm_Horizontal_Fastron_MISC
- added ?: , , F.Cu at (131.6, 39.4)
- added ?: , , F.Cu at (131.6, 108.9)
- added C31: 1µF, Capacitor_THT:C_Disc_D7.5mm_W5.0mm_P5.00mm, F.Cu at (56.0, 111.0)
- added C32: 100µF, Capacitor_THT:CP_Radial_D6.3mm_P2.50mm, F.Cu at (48.3, 112.3)
- added C33: 220µF, Capacitor_THT:CP_Radial_D8.0mm_P5.00mm, F.Cu at (20.6, 31.3)
- added C34: 1µF, Capacitor_THT:C_Disc_D7.5mm_W5.0mm_P5.00mm, F.Cu at (32.0, 35.2)
- added R33: 3k3, Resistor_THT:R_Axial_DIN0207_L6.3mm_D2.5mm_P10.16mm_Horizontal, F.Cu at (17.3, 117.1)
- added R34: 3k3, Resistor_THT:R_Axial_DIN0207_L6.3mm_D2.5mm_P10.16mm_Horizontal, F.Cu at (32.7, 117.3)
- added R35: 3k3, Resistor_THT:R_Axial_DIN0207_L6.3mm_D2.5mm_P10.16mm_Horizontal, F.Cu at (47.7, 125.8)
- added R36: 3k3, Resistor_THT:R_Axial_DIN0207_L6.3mm_D2.5mm_P10.16mm_Horizontal, F.Cu at (39.3, 46.5)
- added R37: 3k3, Resistor_THT:R_Axial_DIN0207_L6.3mm_D2.5mm_P10.16mm_Horizontal, F.Cu at (39.3, 43.1)
- added R38: 1.5, Resistor_THT:R_Axial_DIN0207_L6.3mm_D2.5mm_P10.16mm_Horizontal, F.Cu at (125.4, 18.0)
- added R39: 1.5, Resistor_THT:R_Axial_DIN0207_L6.3mm_D2.5mm_P10.16mm_Horizontal, F.Cu at (128.9, 45.8)
- added R40: 1.5, Resistor_THT:R_Axial_DIN0207_L6.3mm_D2.5mm_P10.16mm_Horizontal, F.Cu at (129.3, 71.0)
- R10, R15, R18: value 1 -> 1.5
- R11, R12, R13, R14, R20, R21, R25, R26: value 1k -> 3k3
- moved R30 339.6 mm to (17.4, 120.7)
- moved R31 323.9 mm to (32.7, 120.9)
- moved R32 309.5 mm to (47.7, 129.2)
- moved C28 297.1 mm to (22.8, 112.1), turned to 180 degrees
- moved R29 283.2 mm to (74.2, 117.1), turned to 180 degrees
- moved C29 281.4 mm to (38.2, 112.2), turned to 180 degrees
- moved C30 266.5 mm to (53.2, 121.1), turned to 180 degrees
- moved R24 262.2 mm to (81.8, 126.5)
- moved R19 254.0 mm to (91.9, 117.2), turned to 180 degrees
- moved C27 250.9 mm to (69.5, 112.6), turned to 180 degrees
- moved R27 238.0 mm to (123.0, 123.8), turned to 180 degrees
- moved C26 235.3 mm to (87.2, 121.8), turned to 180 degrees
- moved C25 235.0 mm to (87.2, 112.6), turned to 180 degrees
- moved R23 233.9 mm to (110.0, 120.1), turned to 180 degrees
- moved R28 232.4 mm to (128.6, 127.1), turned to 90 degrees
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Connections:
- C19 pad 1: HalfVcc -> ADC1_IN4
- C21 pad 1: HalfVcc -> ADC1_IN4
- C24 pad 1: HalfVcc -> ADC1_IN4
- C25 pad 1: Ph1-2_ADC -> ADC1_IN10
- C26 pad 1: Ph1-2_ADC -> ADC2_IN12
- C27 pad 1: Ph1-2_ADC -> ADC3_IN0
- C28 pad 1: Current_Phase_1 -> ADC1_IN11
- C29 pad 1: Current_Phase_2 -> ADC2_IN13
- C30 pad 1: Current_Phase_2 -> ADC3_IN1
- J1 pad 2: Net-(J1-Pin_2) -> +5V
- Q2 pad 1: +5V -> Net-(D1-A)
- Q2 pad 3: Net-(D1-A) -> +5V
- Q5 pad 1: +5V -> Net-(D5-A)
- Q5 pad 3: Net-(D5-A) -> +5V
- Q8 pad 1: +5V -> Net-(D8-A)
- Q8 pad 3: Net-(D8-A) -> +5V
- R13 pad 2: +5V -> +3.3V
- R16 pad 1: OffsetVoltage -> ADC1_IN4
- R18 pad 2: Phase1 -> Phase3
- R19 pad 2: Ph1-2_ADC -> ADC1_IN10
- R2 pad 1: unconnected-(R2-Pad1) -> TIM_CH1
- R22 pad 1: OffsetVoltage -> ADC1_IN4
- R24 pad 2: Ph1-2_ADC -> ADC2_IN12
- R27 pad 1: OffsetVoltage -> ADC1_IN4
- R29 pad 2: Ph1-2_ADC -> ADC3_IN0
- R3 pad 1: unconnected-(R3-Pad1) -> TIM_CH1N
- R30 pad 1: Current_Phase_1 -> ADC1_IN11
- R31 pad 1: Current_Phase_2 -> ADC2_IN13
- R32 pad 1: Current_Phase_2 -> ADC3_IN1
- R4 pad 1: unconnected-(R4-Pad1) -> TIM_CH2
- R5 pad 1: unconnected-(R5-Pad1) -> TIM_CH2N
- R7 pad 1: unconnected-(R7-Pad1) -> TIM_CH3
- R8 pad 1: unconnected-(R8-Pad1) -> TIM_CH3N
- U1 pad CN10_1: (no net) -> unconnected-(U1B-PC9-PadCN10_1)
- U1 pad CN10_11: (no net) -> unconnected-(U1B-PA5-PadCN10_11)
- U1 pad CN10_12: (no net) -> unconnected-(U1B-PA12-PadCN10_12)
- U1 pad CN10_13: (no net) -> ADC2_IN6
- U1 pad CN10_14: (no net) -> unconnected-(U1B-PA11-PadCN10_14)
- U1 pad CN10_15: (no net) -> unconnected-(U1B-PA7-PadCN10_15)
- U1 pad CN10_16: (no net) -> unconnected-(U1B-PB12-PadCN10_16)
- U1 pad CN10_17: (no net) -> unconnected-(U1B-PB6-PadCN10_17)
- U1 pad CN10_19: (no net) -> unconnected-(U1B-PC7-PadCN10_19)
- U1 pad CN10_2: (no net) -> unconnected-(U1B-PC8-PadCN10_2)
- U1 pad CN10_20: (no net) -> GND
- U1 pad CN10_21: (no net) -> TIM_CH2
- U1 pad CN10_22: (no net) -> unconnected-(U1B-PB2-PadCN10_22)
- U1 pad CN10_23: (no net) -> TIM_CH1
- U1 pad CN10_24: (no net) -> unconnected-(U1B-PB1-PadCN10_24)
- U1 pad CN10_25: (no net) -> unconnected-(U1B-PB10-PadCN10_25)
- U1 pad CN10_26: (no net) -> TIM_CH3N
- U1 pad CN10_27: (no net) -> unconnected-(U1B-PB4-PadCN10_27)
- U1 pad CN10_28: (no net) -> TIM_CH2N
- U1 pad CN10_29: (no net) -> unconnected-(U1B-PB5-PadCN10_29)
- U1 pad CN10_3: (no net) -> unconnected-(U1B-PB8-PadCN10_3)
- U1 pad CN10_30: (no net) -> TIM_CH1N
- U1 pad CN10_31: (no net) -> unconnected-(U1B-PB3-PadCN10_31)
- U1 pad CN10_32: (no net) -> unconnected-(U1B-AGND-PadCN10_32)
- U1 pad CN10_33: (no net) -> TIM_CH3
- U1 pad CN10_34: (no net) -> unconnected-(U1B-PC4-PadCN10_34)
- U1 pad CN10_35: (no net) -> unconnected-(U1B-PA2-PadCN10_35)
- U1 pad CN10_37: (no net) -> unconnected-(U1B-PA3-PadCN10_37)
- U1 pad CN10_4: (no net) -> unconnected-(U1B-PC6-PadCN10_4)
- U1 pad CN10_5: (no net) -> unconnected-(U1B-PB9-PadCN10_5)
- U1 pad CN10_6: (no net) -> unconnected-(U1B-PC5-PadCN10_6)
- U1 pad CN10_7: (no net) -> unconnected-(U1B-AVDD-PadCN10_7)
- U1 pad CN10_8: (no net) -> unconnected-(U1B-U5V-PadCN10_8)
- U1 pad CN10_9: (no net) -> GND
- U1 pad CN5_1: (no net) -> unconnected-(U1F-D8-PadCN5_1)
- U1 pad CN5_10: (no net) -> unconnected-(U1F-D15-PadCN5_10)
- U1 pad CN5_2: (no net) -> unconnected-(U1F-D9-PadCN5_2)
- U1 pad CN5_3: (no net) -> unconnected-(U1F-D10-PadCN5_3)
- U1 pad CN5_4: (no net) -> unconnected-(U1F-D11-PadCN5_4)
- U1 pad CN5_5: (no net) -> unconnected-(U1F-D12-PadCN5_5)
- U1 pad CN5_6: (no net) -> unconnected-(U1F-D13-PadCN5_6)
- U1 pad CN5_7: (no net) -> GND
- U1 pad CN5_8: (no net) -> unconnected-(U1F-AREF-PadCN5_8)
- U1 pad CN5_9: (no net) -> unconnected-(U1F-D14-PadCN5_9)
- U1 pad CN6_2: (no net) -> unconnected-(U1C-CN6_IOREF-PadCN6_2)
- U1 pad CN6_3: (no net) -> unconnected-(U1C-CN6_RESET-PadCN6_3)
- U1 pad CN6_4: (no net) -> +3.3V
- U1 pad CN6_5: (no net) -> unconnected-(U1C-CN6_+5V-PadCN6_5)
- U1 pad CN6_6: (no net) -> GND
- U1 pad CN6_7: (no net) -> GND
- U1 pad CN6_8: (no net) -> unconnected-(U1C-CN6_VIN-PadCN6_8)
- U1 pad CN7_16: unconnected-(U1A-CN7_+3V3-PadCN7_16) -> +3.3V
- U1 pad CN7_19: Net-(U1A-CN7_GND-PadCN7_19) -> GND
- U1 pad CN7_20: Net-(U1A-CN7_GND-PadCN7_19) -> GND
- U1 pad CN7_22: Net-(U1A-CN7_GND-PadCN7_19) -> GND
- U1 pad CN7_28: unconnected-(U1A-PA0-PadCN7_28) -> ADC3_IN0
- U1 pad CN7_30: unconnected-(U1A-PA1-PadCN7_30) -> ADC3_IN1
- U1 pad CN7_32: unconnected-(U1A-PA4-PadCN7_32) -> ADC1_IN4
- U1 pad CN7_35: unconnected-(U1A-PC2-PadCN7_35) -> ADC2_IN12
- U1 pad CN7_36: unconnected-(U1A-PC1/PB9-PadCN7_36) -> ADC1_IN11
- U1 pad CN7_37: unconnected-(U1A-PC3-PadCN7_37) -> ADC2_IN13
- U1 pad CN7_38: unconnected-(U1A-PC0/PB8-PadCN7_38) -> ADC1_IN10
- U1 pad CN7_6: unconnected-(U1A-E5V-PadCN7_6) -> Net-(U1A-E5V)
- U1 pad CN7_8: Net-(U1A-CN7_GND-PadCN7_19) -> GND
- U1 pad CN8_1: (no net) -> unconnected-(U1E-A0-PadCN8_1)
- U1 pad CN8_2: (no net) -> unconnected-(U1E-A1-PadCN8_2)
- U1 pad CN8_3: (no net) -> unconnected-(U1E-A2-PadCN8_3)
- U1 pad CN8_4: (no net) -> unconnected-(U1E-A3-PadCN8_4)
- U1 pad CN8_5: (no net) -> unconnected-(U1E-A4-PadCN8_5)
- U1 pad CN8_6: (no net) -> unconnected-(U1E-A5-PadCN8_6)
- U1 pad CN9_1: (no net) -> unconnected-(U1D-D0-PadCN9_1)
- U1 pad CN9_2: (no net) -> unconnected-(U1D-D1-PadCN9_2)
- U1 pad CN9_3: (no net) -> unconnected-(U1D-D2-PadCN9_3)
- U1 pad CN9_4: (no net) -> unconnected-(U1D-D3-PadCN9_4)
- U1 pad CN9_5: (no net) -> unconnected-(U1D-D4-PadCN9_5)
- U1 pad CN9_6: (no net) -> unconnected-(U1D-D5-PadCN9_6)
- U1 pad CN9_7: (no net) -> unconnected-(U1D-D6-PadCN9_7)
- U1 pad CN9_8: (no net) -> unconnected-(U1D-D7-PadCN9_8)
- U2 pad 5: HalfVcc -> ADC1_IN4
- U3 pad 5: HalfVcc -> ADC1_IN4
- U4 pad 3: Phase1 -> Phase3
- U4 pad 5: HalfVcc -> ADC1_IN4
- U5 pad 1: OffsetVoltage -> ADC1_IN4
- U5 pad 2: OffsetVoltage -> ADC1_IN4

Commit message: A bit of clean-up
Parts:
- removed ? (x2): , 
- removed R33, R34, R35: 3k3, Resistor_THT:R_Axial_DIN0207_L6.3mm_D2.5mm_P10.16mm_Horizontal
- R16, R17, R22, R23, R27, R28: value 1k -> 510
- moved R32 16.5 mm to (64.0, 126.6)
- moved C30 16.4 mm to (69.5, 122.0)
- moved R31 3.94 mm to (32.7, 116.9)
- moved R30 3.93 mm to (17.3, 116.7)
Other:
- board outline added: 139.7 x 116.8 mm

Commit message: First Routing
Parts:
- moved R24 10.2 mm to (91.9, 126.3), turned to 180 degrees
Routing:
- net GND: track 0.00 -> 833.0 mm
- net +5V: track 0.00 -> 399.6 mm, vias 0 -> 1
- net ADC1_IN4: track 0.00 -> 202.0 mm, vias 0 -> 1
- net Net-(R30-Pad2): track 0.00 -> 181.9 mm, vias 0 -> 1
- net Net-(R32-Pad2): track 0.00 -> 154.1 mm, vias 0 -> 1
- net Net-(R31-Pad2): track 0.00 -> 144.3 mm, vias 0 -> 1
- net GND1: track 0.00 -> 118.4 mm
- net Phase2: track 0.00 -> 113.7 mm
- net Phase3: track 0.00 -> 110.6 mm, vias 0 -> 1
- net Phase1: track 0.00 -> 104.2 mm
- net ADC1_IN11: track 0.00 -> 79.6 mm
- net TIM_CH3: track 0.00 -> 68.4 mm
- net ADC2_IN13: track 0.00 -> 63.5 mm
- net TIM_CH3N: track 0.00 -> 61.2 mm, vias 0 -> 1
- net Net-(R28-Pad2): track 0.00 -> 58.9 mm
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
Commit message: Generated Gaber files
Other:
- board text added: "5V, GND"
- board text added: "Ph3, Ph2, Ph1"
Changed lines of the file:
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@@
     (property "ki_keywords" "screw terminal")
     (attr through_hole)
-    (fp_text reference "J2" (at 5.05 -4.65 90) (layer "F.SilkS")
+    (fp_text reference "J2" (at -2.119204 -4.810439 90) (layer "F.SilkS")
         (effects (font (size 1 1) (thickness 0.15)))
     )
@@
   (gr_rect (start 12.7 12.7) (end 152.4 129.54)
     (stroke (width 0.1) (type default)) (fill none) (layer "Edge.Cuts"))
+  (gr_text "Ph3, Ph2, Ph1" (at 142.24 30.48 90) (layer "F.SilkS")
+    (effects (font (size 1 1) (thickness 0.15)) (justify left bottom))
+  )
+  (gr_text "5V, GND" (at 22.105535 17.226695 -90) (layer "F.SilkS")
+    (effects (font (size 1 1) (thickness 0.15)) (justify left bottom))
+  )
   (segment (start 106.679999 27.914127) (end 108.240136 27.914127) (width 0.5) (layer "B.Cu") (net 1))
   (segment (start 99.856666 17.724127) (end 99.906666 17.774127) (width 0.5) (layer "B.Cu") (net 1))
